File: KiCad_Traffic_Light_Controller/KiCad_Traffic_Light_Controller.kicad_pcb (KiCad board)
At the start: 2 copper layers, 193.3 x 100.6 mm, 65 parts, among them J1 Conn_02x08_Odd_Even, J2 Conn_02x08_Odd_Even, J3 Conn_02x05_Odd_Even, J4 +5V, SW1 RST, SW2 OVR, SW3 EN, U1 SM420561N, U2 SM420561N, U3 LM1117DT-3.3

Commit message: clutch
Parts:
- removed G***: LOGO, my_footprints:Gyronix-logo-10mm x 10mm
- moved H1 5.88 mm to (210.3, 121.4)
- moved H3 5.77 mm to (210.3, 41.1)
- moved H2 4.89 mm to (104.6, 41.1)
- moved C3 2.74 mm to (205.7, 102.9), turned to 180 degrees
- moved SW1 2.74 mm to (198.4, 100.3)
- moved C2 2.65 mm to (188.7, 102.9), turned to 180 degrees
- moved C5 2.54 mm to (173.5, 102.9), turned to 180 degrees
- moved SW2 2.41 mm to (182.6, 97.3)
- moved SW3 2.29 mm to (167.4, 97.3)
- moved D12 2.27 mm to (205.7, 98.8), turned to 180 degrees
- moved H4 2.27 mm to (104.6, 121.4)
- moved D11 2.17 mm to (188.7, 98.8), turned to 180 degrees
- moved D13 2.03 mm to (173.5, 98.8), turned to 180 degrees
- moved R29 1.83 mm to (205.7, 94.7)
- moved R28 1.70 mm to (188.7, 94.7), turned to 180 degrees
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Connections:
- C3 pad 1: Net-(D12-K) -> /RST
- D12 pad 1: Net-(D12-K) -> /RST
Routing:
- net GND: track 174.0 -> 444.0 mm, vias 0 -> 4
- net /+3.3V: track 34.8 -> 256.2 mm, vias 0 -> 4
- net /EN: track 10.5 -> 142.3 mm
- net /RST: track 13.3 -> 133.3 mm, vias 0 -> 2
- net /OVR: track 7.47 -> 124.6 mm, vias 0 -> 2
- net /NS_HEX_A: track 11.2 -> 105.2 mm
- net /NS_HEX_B: track 8.82 -> 93.7 mm
- net /EW_HEX_D: track 0.00 -> 79.6 mm
- net /EW_HEX_C: track 0.00 -> 73.1 mm
- net /EW_HEX_DP: track 0.00 -> 66.7 mm, vias 0 -> 1
- net /EW_HEX_E: track 11.4 -> 70.1 mm
- net /+5V: track 26.8 -> 82.0 mm
- net /NS_HEX_DP: track 0.00 -> 54.8 mm, vias 0 -> 1
- net /EWP_RED: track 8.38 -> 62.7 mm
- net /NSP_RED: track 13.5 -> 63.4 mm
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Other:
- board size 193.3 x 100.6 mm -> 111.8 x 86.4 mm

Commit message: final
Parts:
- added REF**: KiCad-Logo2_5mm_SilkScreen, Symbol:KiCad-Logo2_5mm_SilkScreen, B.Cu at (196.8, 116.3)
- moved H2 1.27 mm to (104.6, 39.9)
- moved H3 1.27 mm to (210.3, 39.9)
Routing:
- net /+3.3V: vias 4 -> 3
Other:
- board size 111.8 x 86.4 mm -> 111.8 x 87.6 mm
- board text added: "Computer Engineering Technology S09-A 2026 TUPV"
